File: examples/555-astable/555-astable.kicad_pcb (KiCad board)
At the start: 2 copper layers, 0 parts

Commit message: Validate PCB layout pipeline end-to-end on all 3 example boards
Phase 3 validation: synced, placed, routed (Freerouting), DRC'd, and
exported manufacturing files for 555-astable, opamp-divider, and
esp32c3-breakout. All 3 reach 0 DRC errors, gerbers/drill/PDF exported
to examples/*/gerbers/.

Fix docs/FREEROUTING_GUIDE.md: the documented v2.0.1 jar URL is a dead
release, and more importantly v2.2.0+ requires a newer JDK than the
documented "Java 21+" (confirmed via UnsupportedClassVersionError,
including with the guide's own pinned Docker image). Repin to v2.1.0,
the newest release confirmed to run on Java 21.

Document 3 more field-tested tool/environment gaps in
docs/KNOWN_ISSUES.md (#10-12): sync_schematic_to_board can partially
persist on a save-guard conflict; suggest_placement can hang a
footprint off the board edge while check_courtyard_overlaps reports
clean, inconsistently even for identical input, and a 2-pin THT part's
position is its pad-1 anchor rather than its body center; some library
footprints need finer hole tolerances than a board's default design
rules. Cross-referenced from docs/PCB_DESIGN_WORKFLOW.md.
Parts:
- added C1: 100nF, Capacitor_THT:C_Disc_D5.0mm_W2.5mm_P5.00mm, F.Cu at (6.63, 17.5)
- added C2: 10nF, Capacitor_THT:C_Disc_D5.0mm_W2.5mm_P5.00mm, F.Cu at (6.85, 20.9)
- added D1: LED, LED_THT:LED_D5.0mm, F.Cu at (10.4, 26.0)
- added R1: 10k, Resistor_THT:R_Axial_DIN0207_L6.3mm_D2.5mm_P10.16mm_Horizontal, F.Cu at (35.0, 12.0)
- added R2: 10k, Resistor_THT:R_Axial_DIN0207_L6.3mm_D2.5mm_P10.16mm_Horizontal, F.Cu at (35.0, 26.0)
- added R3: 330, Resistor_THT:R_Axial_DIN0207_L6.3mm_D2.5mm_P10.16mm_Horizontal, F.Cu at (2.67, 13.0)
- added U1: NE555P, Package_DIP:DIP-8_W7.62mm, F.Cu at (13.2, 13.6)
Routing:
- net DISCH: track 0.00 -> 58.3 mm
- net TH_TR: track 0.00 -> 43.4 mm
- net VCC: track 0.00 -> 35.0 mm
- net LED_A: track 0.00 -> 26.3 mm
- net CTRL: track 0.00 -> 16.8 mm
- net GND: track 0.00 -> 13.8 mm
- net OUT: track 0.00 -> 12.4 mm
Other:
- board outline added: 50 x 40 mm
