File: examples/esp32c3-breakout/esp32c3-breakout.kicad_pcb (KiCad board)
At the start: 2 copper layers, 0 parts

Commit message: Validate PCB layout pipeline end-to-end on all 3 example boards
Phase 3 validation: synced, placed, routed (Freerouting), DRC'd, and
exported manufacturing files for 555-astable, opamp-divider, and
esp32c3-breakout. All 3 reach 0 DRC errors, gerbers/drill/PDF exported
to examples/*/gerbers/.

Fix docs/FREEROUTING_GUIDE.md: the documented v2.0.1 jar URL is a dead
release, and more importantly v2.2.0+ requires a newer JDK than the
documented "Java 21+" (confirmed via UnsupportedClassVersionError,
including with the guide's own pinned Docker image). Repin to v2.1.0,
the newest release confirmed to run on Java 21.

Document 3 more field-tested tool/environment gaps in
docs/KNOWN_ISSUES.md (#10-12): sync_schematic_to_board can partially
persist on a save-guard conflict; suggest_placement can hang a
footprint off the board edge while check_courtyard_overlaps reports
clean, inconsistently even for identical input, and a 2-pin THT part's
position is its pad-1 anchor rather than its body center; some library
footprints need finer hole tolerances than a board's default design
rules. Cross-referenced from docs/PCB_DESIGN_WORKFLOW.md.
Parts:
- added C1: 100nF, Capacitor_THT:C_Disc_D5.0mm_W2.5mm_P5.00mm, F.Cu at (8.13, 21.6)
- added J1: UART, Connector_PinHeader_2.54mm:PinHeader_1x04_P2.54mm_Vertical, F.Cu at (15.0, 17.6)
- added R1: 10k, Resistor_THT:R_Axial_DIN0207_L6.3mm_D2.5mm_P10.16mm_Horizontal, F.Cu at (16.5, 13.0)
- added SW1: RESET, Button_Switch_THT:SW_PUSH_6mm, F.Cu at (9.30, 31.6)
- added SW2: BOOT, Button_Switch_THT:SW_PUSH_6mm, F.Cu at (6.26, 9.22)
- added U1: ESP32-C3-WROOM-02, RF_Module:ESP32-C3-WROOM-02, F.Cu at (32.6, 22.5)
Routing:
- net GND: track 0.00 -> 82.0 mm
- net EN: track 0.00 -> 60.3 mm
- net UART_TX: track 0.00 -> 44.3 mm, vias 0 -> 1
- net BOOT: track 0.00 -> 39.1 mm, vias 0 -> 1
- net UART_RX: track 0.00 -> 38.0 mm, vias 0 -> 1
- net VCC: track 0.00 -> 24.8 mm
Other:
- board outline added: 60 x 50 mm
